Commit message: pato changes

File: robutler_description/urdf/robutler.urdf.xacro (robot description, xacro)
@@ -161,8 +161,63 @@
     </inertial>
   </link>
+  <!-- Connect the head to the base -->
+  <link name="head">
+    <visual>
+      <geometry>
+        <sphere radius="0.04"/>
+      </geometry>
+      <material name="turquoise"/>
+    </visual>
+  </link>
+  <joint name="head_swivel" type="fixed">
+    <parent link="camera_to_base"/>
+    <child link="head"/>
+    <origin xyz="0 0 0.5"/>
+  </joint>
+  <link name="box">
+    <visual>
+      <geometry>
+        <box size="0.03 0.03 0.03"/>
+      </geometry>
+      <material name="yellow"/>
+    </visual>
+  </link>
+  <joint name="tobox" type="fixed">
+    <parent link="head"/>
+    <child link="box"/>
+    <origin xyz="0.04 0 0"/>
+  </joint>
+  <link name="box2">
+    <visual>
+      <geometry>
+        <box size="0.04 0.02 0.02"/>
+      </geometry>
+      <material name="yellow"/>
+    </visual>
+  </link>
+  <joint name="tobox2" type="fixed">
+    <parent link="head"/>
+    <child link="box2"/>
+    <origin xyz="0.06 0 0"/>
+  </joint>
+  <!-- Connect Camera to the base -->
+  <link name="camera_to_base">
+    <visual>
+      <geometry>
+        <cylinder length="1" radius="0.02"/>
+      </geometry>
+      <material name="turquoise"/>
+    </visual>
+  </link>
+  <joint name="camera_to_base_joint" type="fixed">
+    <!-- <origin xyz="0.073 -0.011 0.084" rpy="0 0 0"/> -->
+    <origin xyz="0.033 0 0.5" rpy="0 0 0"/>
+    <parent link="base_link"/>
+    <child link="camera_to_base"/>
+  </joint>
   <joint name="camera_joint" type="fixed">
     <!-- <origin xyz="0.073 -0.011 0.084" rpy="0 0 0"/> -->
-    <origin xyz="0.073 -0.011 1" rpy="0 0 0"/>
-    <parent link="base_link"/>
+    <origin xyz="0 0 0.5" rpy="0 0 0"/>
+    <parent link="camera_to_base"/>
     <child link="camera_link"/>
   </joint>

Commit message: camera position fixed

File: robutler_description/urdf/robutler.urdf.xacro (robot description, xacro)
@@ -199,5 +199,5 @@
     <parent link="head"/>
     <child link="box2"/>
-    <origin xyz="0.06 0 0"/>
+    <origin xyz="0.07 0 0"/>
   </joint>
   <!-- Connect Camera to the base -->
@@ -218,5 +218,5 @@
   <joint name="camera_joint" type="fixed">
     <!-- <origin xyz="0.073 -0.011 0.084" rpy="0 0 0"/> -->
-    <origin xyz="0 0 0.5" rpy="0 0 0"/>
+    <origin xyz="0.11 0 0.5" rpy="0 0 0"/>
     <parent link="camera_to_base"/>
     <child link="camera_link"/>

Commit message: robot with claw to get objects -fk how it works now

File: robutler_description/urdf/robutler.urdf.xacro (robot description, xacro)
@@ -242,3 +242,74 @@
   </joint>
   <link name="camera_rgb_optical_frame"/>
+  <!-- Arm claw -->
+  <!-- Connect CameraBase to the claw -->
+  <link name="pole_to_claw">
+    <visual>
+      <geometry>
+        <cylinder length="0.1" radius="0.012"/>
+      </geometry>
+      <material name="turquoise"/>
+    </visual>
+  </link>
+  <joint name="pole_to_claw_joint" type="fixed">
+    <!-- <origin xyz="0.073 -0.011 0.084" rpy="0 0 0"/> -->
+    <origin xyz="0.05 0 -0.35" rpy="0 1.57075 0"/>
+    <parent link="camera_to_base"/>
+    <child link="pole_to_claw"/>
+  </joint>
+  <link name="claw_right_first">
+    <visual>
+      <geometry>
+        <cylinder length="0.05" radius="0.01"/>
+      </geometry>
+      <material name="turquoise"/>
+    </visual>
+  </link>
+  <joint name="pole_to_claw_right_first_joint" type="fixed">
+    <!-- <origin xyz="0.073 -0.011 0.084" rpy="0 0 0"/> -->
+    <origin xyz="0 -0.02 0.055" rpy="0.8 0 0"/>
+    <parent link="pole_to_claw"/>
+    <child link="claw_right_first"/>
+  </joint>
+  <link name="claw_right_second">
+    <visual>
+      <geometry>
+        <cylinder length="0.03" radius="0.01"/>
+      </geometry>
+      <material name="turquoise"/>
+    </visual>
+  </link>
+  <joint name="pole_to_claw_right_second_joint" type="fixed">
+    <!-- <origin xyz="0.073 -0.011 0.084" rpy="0 0 0"/> -->
+    <origin xyz="0 0.01 ${0.0148 + 0.01}" rpy="1.57075 0 0"/>
+    <parent link="claw_right_first"/>
+    <child link="claw_right_second"/>
+  </joint>
+  <link name="claw_left_first">
+    <visual>
+      <geometry>
+        <cylinder length="0.05" radius="0.01"/>
+      </geometry>
+      <material name="turquoise"/>
+    </visual>
+  </link>
+  <joint name="pole_to_claw_left_first_joint" type="fixed">
+    <!-- <origin xyz="0.073 -0.011 0.084" rpy="0 0 0"/> -->
+    <origin xyz="0 0.02 0.055" rpy="-0.8 0 0"/>
+    <parent link="pole_to_claw"/>
+    <child link="claw_left_first"/>
+  </joint>
+  <link name="claw_left_second">
+    <visual>
+      <geometry>
+        <cylinder length="0.03" radius="0.01"/>
+      </geometry>
+      <material name="turquoise"/>
+    </visual>
+  </link>
+  <joint name="pole_to_claw_left_second_joint" type="fixed">
+    <origin xyz="0 -0.01 ${0.0148 + 0.01}" rpy="-1.57075 0 0"/>
+    <parent link="claw_left_first"/>
+    <child link="claw_left_second"/>
+  </joint>
 </robot>
