Commit message: claw works but not in pyrhon stillç

File: robutler_description/urdf/robutler.gazebo.xacro (robot description, xacro)
@@ -4,6 +4,52 @@
   <xacro:arg name="camera_visual" default="false"/>
   <xacro:arg name="imu_visual"    default="false"/>
+  <gazebo>
+    <plugin name="gazebo_ros_control" filename="libgazebo_ros_control.so">
+      <robotNamespace>/robutler</robotNamespace>
+    </plugin>
+  </gazebo>
   <gazebo reference="base_link">
     <!-- <material>Gazebo/DarkGrey</material> -->
+    <material>Gazebo/Turquoise</material>
+  </gazebo>
+  <gazebo reference="pole_to_middle">
+    <material>Gazebo/Turquoise</material>
+  </gazebo>
+  <gazebo reference="base_middle">
+    <material>Gazebo/Turquoise</material>
+  </gazebo>
+  <gazebo reference="box2">
+    <material>Gazebo/Yellow</material>
+  </gazebo>
+  <gazebo reference="box">
+    <material>Gazebo/Yellow</material>
+  </gazebo>
+  <gazebo reference="head">
+    <material>Gazebo/Turquoise</material>
+  </gazebo>
+  <gazebo reference="camera_to_base">
+    <material>Gazebo/Turquoise</material>
+  </gazebo>
+  <gazebo reference="camera_base_to_base">
+    <material>Gazebo/Turquoise</material>
+  </gazebo>
+  <gazebo reference="claw_right_second">
+    <mu1>0.1</mu1>
+    <mu2>0.1</mu2>
+    <kp>500000.0</kp>
+    <kd>10.0</kd>
+    <minDepth>0.001</minDepth>
+    <maxVel>0.1</maxVel>
+    <fdir1>1 0 0</fdir1>
+    <material>Gazebo/Turquoise</material>
+  </gazebo>
+  <gazebo reference="claw_left_second">
+    <mu1>0.1</mu1>
+    <mu2>0.1</mu2>
+    <kp>500000.0</kp>
+    <kd>10.0</kd>
+    <minDepth>0.001</minDepth>
+    <maxVel>0.1</maxVel>
+    <fdir1>1 0 0</fdir1>
     <material>Gazebo/Turquoise</material>
   </gazebo>
@@ -55,4 +101,11 @@
     <material>Gazebo/Grey</material>
   </gazebo>
+  <!-- <gazebo>
+    <plugin name="JointStatePublisher" filename="libJointStatePublisher.so">
+      <joint>pole_to_claw_right_second_joint</joint>
+      <joint>pole_to_claw_left_second_joint</joint>
+      <publish_selected_only>true</publish_selected_only>
+    </plugin>
+  </gazebo> -->
   <gazebo>
     <plugin name="turtlebot3_waffle_pi_controller" filename="libgazebo_ros_diff_drive.so">

File: robutler_description/urdf/robutler.urdf.xacro (robot description, xacro)
@@ -242,4 +242,41 @@
   </joint>
   <link name="camera_rgb_optical_frame"/>
+  <!-- Weight distribution -->
+  <link name="base_middle">
+    <visual>
+      <geometry>
+        <cylinder length="0.25" radius="0.02"/>
+      </geometry>
+      <material name="turquoise"/>
+    </visual>
+    <collision>
+      <origin xyz="0 0 0" rpy="0 0 0"/>
+      <geometry>
+        <cylinder length="0.25" radius="0.02"/>
+      </geometry>
+    </collision>
+    <inertial>
+      <mass value="0.5" />
+      <inertia ixx="0.4" ixy="0.0" ixz="0.0" iyy="0.4" iyz="0.0" izz="0.2"/>
+    </inertial>
+  </link>
+  <joint name="base_middle_joint" type="fixed">
+    <origin xyz="-0.145 0 0.15" rpy="0 0 0"/>
+    <parent link="base_link"/>
+    <child link="base_middle"/>
+  </joint>
+  <link name="pole_to_middle">
+    <visual>
+      <geometry>
+        <cylinder length="0.178" radius="0.02"/>
+      </geometry>
+      <material name="turquoise"/>
+    </visual>
+  </link>
+  <joint name="pole_to_middle_joint" type="fixed">
+    <origin xyz="0 0 0.089" rpy="1.57075 0 0"/>
+    <parent link="base_middle"/>
+    <child link="pole_to_middle"/>
+  </joint>
   <!-- Arm claw -->
   <!-- Connect CameraBase to the claw -->
@@ -254,5 +291,5 @@
   <joint name="pole_to_claw_joint" type="fixed">
     <!-- <origin xyz="0.073 -0.011 0.084" rpy="0 0 0"/> -->
-    <origin xyz="0.05 0 -0.35" rpy="0 1.57075 0"/>
+    <origin xyz="0.05 0 -0.25" rpy="0 1.57075 0"/>
     <parent link="camera_to_base"/>
     <child link="pole_to_claw"/>
@@ -265,4 +302,8 @@
       <material name="turquoise"/>
     </visual>
+    <inertial>
+        <mass value="0.18" />
+        <inertia ixx="0.0002835" ixy="0.0" ixz="0.0" iyy="0.0002835" iyz="0.0" izz="0.000324" />
+    </inertial>
   </link>
   <joint name="pole_to_claw_right_first_joint" type="fixed">
@@ -279,10 +320,20 @@
       <material name="turquoise"/>
     </visual>
-  </link>
-  <joint name="pole_to_claw_right_second_joint" type="fixed">
-    <!-- <origin xyz="0.073 -0.011 0.084" rpy="0 0 0"/> -->
+    <collision>
+      <origin xyz="0 0 0" rpy="0 0 0"/>
+      <geometry>
+        <cylinder length="0.018" radius="0.033"/>
+      </geometry>
+    </collision>
+    <inertial>
+      <mass value="0.04" />
+      <inertia ixx="0.4" ixy="0.0" ixz="0.0" iyy="0.4" iyz="0.0" izz="0.2"/>
+    </inertial>
+  </link>
+  <joint name="pole_to_claw_right_second_joint" type="continuous">
     <origin xyz="0 0.01 ${0.0148 + 0.01}" rpy="1.57075 0 0"/>
     <parent link="claw_right_first"/>
     <child link="claw_right_second"/>
+    <dynamics damping="0.7"/>
   </joint>
   <link name="claw_left_first">
@@ -293,4 +344,8 @@
       <material name="turquoise"/>
     </visual>
+    <inertial>
+      <mass value="0.18" />
+      <inertia ixx="0.0002835" ixy="0.0" ixz="0.0" iyy="0.0002835" iyz="0.0" izz="0.000324" />
+    </inertial>
   </link>
   <joint name="pole_to_claw_left_first_joint" type="fixed">
@@ -307,9 +362,42 @@
       <material name="turquoise"/>
     </visual>
-  </link>
-  <joint name="pole_to_claw_left_second_joint" type="fixed">
+    <collision>
+      <origin xyz="0 0 0" rpy="0 0 0"/>
+      <geometry>
+        <cylinder length="0.018" radius="0.033"/>
+      </geometry>
+    </collision>
+    <inertial>
+      <mass value="0.04" />
+      <inertia ixx="0.4" ixy="0.0" ixz="0.0" iyy="0.4" iyz="0.0" izz="0.2"/>
+      </inertial>
+  </link>
+  <joint name="pole_to_claw_left_second_joint" type="continuous">
     <origin xyz="0 -0.01 ${0.0148 + 0.01}" rpy="-1.57075 0 0"/>
     <parent link="claw_left_first"/>
     <child link="claw_left_second"/>
-  </joint>
+    <dynamics damping="0.7"/>
+  </joint>
+  <!-- transmission -->
+  <transmission name="right_claw">
+    <type>transmission_interface/SimpleTransmission</type>
+    <actuator name="right_claw_actuator">
+      <mechanicalReduction>20</mechanicalReduction>
+      <hardwareInterface>hardware_interface/EffortJointInterface</hardwareInterface>
+    </actuator>
+    <joint name="pole_to_claw_right_second_joint">
+      <hardwareInterface>hardware_interface/EffortJointInterface</hardwareInterface>
+    </joint>
+  </transmission>
+  <!-- transmission -->
+  <transmission name="left_claw">
+    <type>transmission_interface/SimpleTransmission</type>
+    <actuator name="left_claw_actuator">
+      <mechanicalReduction>20</mechanicalReduction>
+      <hardwareInterface>hardware_interface/EffortJointInterface</hardwareInterface>
+    </actuator>
+    <joint name="pole_to_claw_left_second_joint">
+      <hardwareInterface>hardware_interface/EffortJointInterface</hardwareInterface>
+    </joint>
+  </transmission>
 </robot>
